File: VSource.kicad_pcb (KiCad board)
At the start: 2 copper layers, 50 x 50 mm, 12 parts, among them J1 - +, J2 - +, U1 LM317_TO-220

Commit message: 5v output
Parts:
- removed the C1 at (169.5, 73.0)
- removed the C2 at (162.0, 82.0)
- removed the C3 at (151.5, 60.0)
- removed the D1 at (151.9, 74.0)
- removed the D2 at (146.8, 87.0)
- removed the D3 at (141.0, 73.0)
- removed the J1 at (137.0, 54.0)
- removed the J2 at (171.9, 59.0)
- removed the R1 at (132.8, 96.0)
- removed the R2 at (153.4, 96.0)
- removed the RV1 at (173.0, 96.0)
- removed the U1 at (134.0, 90.1)
- added C1: 1uF, Capacitor_THT:CP_Radial_Tantal_D4.5mm_P2.50mm, F.Cu at (47.5, 172.7)
- added C1: 1uF, Capacitor_THT:CP_Radial_Tantal_D4.5mm_P2.50mm, F.Cu at (233.0, 116.7)
- added C1: 1uF, Capacitor_THT:CP_Radial_Tantal_D4.5mm_P2.50mm, F.Cu at (234.0, 50.7)
- added C1: 1uF, Capacitor_THT:CP_Radial_Tantal_D4.5mm_P2.50mm, F.Cu at (139.5, 117.2)
- added C1: 1uF, Capacitor_THT:CP_Radial_Tantal_D4.5mm_P2.50mm, F.Cu at (142.1, 51.6)
- added C1: 1uF, Capacitor_THT:CP_Radial_Tantal_D4.5mm_P2.50mm, F.Cu at (48.0, 52.2)
- added C1: 1uF, Capacitor_THT:CP_Radial_Tantal_D4.5mm_P2.50mm, F.Cu at (48.0, 117.2)
- added C2: 10uF, Capacitor_THT:CP_Radial_D4.0mm_P2.00mm, F.Cu at (147.5, 119.5)
- added C2: 10uF, Capacitor_THT:CP_Radial_D4.0mm_P2.00mm, F.Cu at (55.5, 175.0)
- added C2: 10uF, Capacitor_THT:CP_Radial_D4.0mm_P2.00mm, F.Cu at (242.0, 53.0)
- added C2: 10uF, Capacitor_THT:CP_Radial_D4.0mm_P2.00mm, F.Cu at (56.0, 54.5)
- added C2: 10uF, Capacitor_THT:CP_Radial_D4.0mm_P2.00mm, F.Cu at (241.0, 119.0)
- added C2: 10uF, Capacitor_THT:CP_Radial_D4.0mm_P2.00mm, F.Cu at (56.0, 119.5)
- added C2: 10uF, Capacitor_THT:CP_Radial_D4.0mm_P2.00mm, F.Cu at (150.1, 53.9)
- added C3: 4700uF, Capacitor_THT:CP_Radial_D18.0mm_P7.50mm, F.Cu at (48.0, 39.5)
- added C3: 4700uF, Capacitor_THT:CP_Radial_D18.0mm_P7.50mm, F.Cu at (139.5, 104.5)
- added C3: 4700uF, Capacitor_THT:CP_Radial_D18.0mm_P7.50mm, F.Cu at (47.5, 160.0)
- added C3: 4700uF, Capacitor_THT:CP_Radial_D18.0mm_P7.50mm, F.Cu at (48.0, 104.5)
- added C3: 4700uF, Capacitor_THT:CP_Radial_D18.0mm_P7.50mm, F.Cu at (142.1, 38.9)
- added C3: 4700uF, Capacitor_THT:CP_Radial_D18.0mm_P7.50mm, F.Cu at (233.0, 104.0)
- added C3: 4700uF, Capacitor_THT:CP_Radial_D18.0mm_P7.50mm, F.Cu at (234.0, 38.0)
- added C4: 0.33uF, Capacitor_THT:CP_Radial_Tantal_D5.0mm_P2.50mm, F.Cu at (243.8, 27.0)
- added C4: 0.33uF, Capacitor_THT:CP_Radial_Tantal_D5.0mm_P2.50mm, F.Cu at (151.9, 27.9)
- added C4: 0.33uF, Capacitor_THT:CP_Radial_Tantal_D5.0mm_P2.50mm, F.Cu at (149.3, 93.5)
- added C4: 0.33uF, Capacitor_THT:CP_Radial_Tantal_D5.0mm_P2.50mm, F.Cu at (57.8, 93.5)
- added C4: 0.33uF, Capacitor_THT:CP_Radial_Tantal_D5.0mm_P2.50mm, F.Cu at (242.8, 93.0)
- added C4: 0.33uF, Capacitor_THT:CP_Radial_Tantal_D5.0mm_P2.50mm, F.Cu at (57.3, 149.0)
- added C4: 0.33uF, Capacitor_THT:CP_Radial_Tantal_D5.0mm_P2.50mm, F.Cu at (57.8, 28.5)
- added C5: 0.1uF, Capacitor_THT:CP_Radial_Tantal_D5.0mm_P2.50mm, F.Cu at (150.0, 110.5)
- added C5: 0.1uF, Capacitor_THT:CP_Radial_Tantal_D5.0mm_P2.50mm, F.Cu at (58.5, 110.5)
- added C5: 0.1uF, Capacitor_THT:CP_Radial_Tantal_D5.0mm_P2.50mm, F.Cu at (58.5, 45.5)
- added C5: 0.1uF, Capacitor_THT:CP_Radial_Tantal_D5.0mm_P2.50mm, F.Cu at (244.5, 44.0)
- added C5: 0.1uF, Capacitor_THT:CP_Radial_Tantal_D5.0mm_P2.50mm, F.Cu at (243.5, 110.0)
- added C5: 0.1uF, Capacitor_THT:CP_Radial_Tantal_D5.0mm_P2.50mm, F.Cu at (152.6, 44.9)
- added C5: 0.1uF, Capacitor_THT:CP_Radial_Tantal_D5.0mm_P2.50mm, F.Cu at (58.0, 166.0)
- added D1: 1N4007, Diode_THT:D_DO-41_SOD81_P10.16mm_Horizontal, F.Cu at (129.6, 131.5)
- added D1: 1N4007, Diode_THT:D_DO-41_SOD81_P10.16mm_Horizontal, F.Cu at (223.1, 131.0)
- added D1: 1N4007, Diode_THT:D_DO-41_SOD81_P10.16mm_Horizontal, F.Cu at (224.1, 65.0)
- added D1: 1N4007, Diode_THT:D_DO-41_SOD81_P10.16mm_Horizontal, F.Cu at (38.1, 131.5)
- added D1: 1N4007, Diode_THT:D_DO-41_SOD81_P10.16mm_Horizontal, F.Cu at (132.2, 65.9)
- added D1: 1N4007, Diode_THT:D_DO-41_SOD81_P10.16mm_Horizontal, F.Cu at (37.6, 187.0)
- added D1: 1N4007, Diode_THT:D_DO-41_SOD81_P10.16mm_Horizontal, F.Cu at (38.1, 66.5)
- added D2: 1N4007, Diode_THT:D_DO-41_SOD81_P10.16mm_Horizontal, F.Cu at (59.5, 70.6)
- added D2: 1N4007, Diode_THT:D_DO-41_SOD81_P10.16mm_Horizontal, F.Cu at (151.0, 135.6)
- added D2: 1N4007, Diode_THT:D_DO-41_SOD81_P10.16mm_Horizontal, F.Cu at (59.0, 191.1)
- added D2: 1N4007, Diode_THT:D_DO-41_SOD81_P10.16mm_Horizontal, F.Cu at (153.6, 70.0)
- added D2: 1N4007, Diode_THT:D_DO-41_SOD81_P10.16mm_Horizontal, F.Cu at (244.5, 135.1)
- added D2: 1N4007, Diode_THT:D_DO-41_SOD81_P10.16mm_Horizontal, F.Cu at (245.5, 69.1)
- added D2: 1N4007, Diode_THT:D_DO-41_SOD81_P10.16mm_Horizontal, F.Cu at (59.5, 135.6)
- added D3: B40C3x00-2200A, Diode_THT:Diode_Bridge_Round_D9.0mm, F.Cu at (120.1, 43.9)
- added D3: B40C3x00-2200A, Diode_THT:Diode_Bridge_Round_D9.0mm, F.Cu at (26.0, 44.5)
- added D3: B40C3x00-2200A, Diode_THT:Diode_Bridge_Round_D9.0mm, F.Cu at (25.5, 165.0)
- added D3: B40C3x00-2200A, Diode_THT:Diode_Bridge_Round_D9.0mm, F.Cu at (212.0, 43.0)
- added D3: B40C3x00-2200A, Diode_THT:Diode_Bridge_Round_D9.0mm, F.Cu at (211.0, 109.0)
- added D3: B40C3x00-2200A, Diode_THT:Diode_Bridge_Round_D9.0mm, F.Cu at (26.0, 109.5)
- added D3: B40C3x00-2200A, Diode_THT:Diode_Bridge_Round_D9.0mm, F.Cu at (117.5, 109.5)
- added J1: - +, TerminalBlock_MetzConnect:TerminalBlock_MetzConnect_Type055_RT01502HDWU_1x02_P5.00mm_Horizontal, F.Cu at (213.0, 26.5)
- added J1: - +, TerminalBlock_MetzConnect:TerminalBlock_MetzConnect_Type055_RT01502HDWU_1x02_P5.00mm_Horizontal, F.Cu at (26.5, 148.5)
- added J1: - +, TerminalBlock_MetzConnect:TerminalBlock_MetzConnect_Type055_RT01502HDWU_1x02_P5.00mm_Horizontal, F.Cu at (121.1, 27.4)
- added J1: - +, TerminalBlock_MetzConnect:TerminalBlock_MetzConnect_Type055_RT01502HDWU_1x02_P5.00mm_Horizontal, F.Cu at (118.5, 93.0)
- added J1: - +, TerminalBlock_MetzConnect:TerminalBlock_MetzConnect_Type055_RT01502HDWU_1x02_P5.00mm_Horizontal, F.Cu at (212.0, 92.5)
- added J1: - +, TerminalBlock_MetzConnect:TerminalBlock_MetzConnect_Type055_RT01502HDWU_1x02_P5.00mm_Horizontal, F.Cu at (27.0, 93.0)
- added J1: - +, TerminalBlock_MetzConnect:TerminalBlock_MetzConnect_Type055_RT01502HDWU_1x02_P5.00mm_Horizontal, F.Cu at (27.0, 28.0)
- added J2: - +, TerminalBlock_MetzConnect:TerminalBlock_MetzConnect_Type055_RT01502HDWU_1x02_P5.00mm_Horizontal, F.Cu at (66.5, 53.5)
- added J2: - +, TerminalBlock_MetzConnect:TerminalBlock_MetzConnect_Type055_RT01502HDWU_1x02_P5.00mm_Horizontal, F.Cu at (158.0, 118.5)
- added J2: - +, TerminalBlock_MetzConnect:TerminalBlock_MetzConnect_Type055_RT01502HDWU_1x02_P5.00mm_Horizontal, F.Cu at (66.0, 174.0)
- added J2: - +, TerminalBlock_MetzConnect:TerminalBlock_MetzConnect_Type055_RT01502HDWU_1x02_P5.00mm_Horizontal, F.Cu at (66.5, 118.5)
- added J2: - +, TerminalBlock_MetzConnect:TerminalBlock_MetzConnect_Type055_RT01502HDWU_1x02_P5.00mm_Horizontal, F.Cu at (251.5, 118.0)
- added J2: - +, TerminalBlock_MetzConnect:TerminalBlock_MetzConnect_Type055_RT01502HDWU_1x02_P5.00mm_Horizontal, F.Cu at (160.6, 52.9)
- added J2: - +, TerminalBlock_MetzConnect:TerminalBlock_MetzConnect_Type055_RT01502HDWU_1x02_P5.00mm_Horizontal, F.Cu at (252.5, 52.0)
- added J3: - +, TerminalBlock_MetzConnect:TerminalBlock_MetzConnect_Type055_RT01502HDWU_1x02_P5.00mm_Horizontal, F.Cu at (66.5, 98.0)
- added J3: - +, TerminalBlock_MetzConnect:TerminalBlock_MetzConnect_Type055_RT01502HDWU_1x02_P5.00mm_Horizontal, F.Cu at (158.0, 98.0)
- added J3: - +, TerminalBlock_MetzConnect:TerminalBlock_MetzConnect_Type055_RT01502HDWU_1x02_P5.00mm_Horizontal, F.Cu at (251.5, 97.5)
- added J3: - +, TerminalBlock_MetzConnect:TerminalBlock_MetzConnect_Type055_RT01502HDWU_1x02_P5.00mm_Horizontal, F.Cu at (66.5, 33.0)
- added J3: - +, TerminalBlock_MetzConnect:TerminalBlock_MetzConnect_Type055_RT01502HDWU_1x02_P5.00mm_Horizontal, F.Cu at (160.6, 32.4)
- added J3: - +, TerminalBlock_MetzConnect:TerminalBlock_MetzConnect_Type055_RT01502HDWU_1x02_P5.00mm_Horizontal, F.Cu at (66.0, 153.5)
- added J3: - +, TerminalBlock_MetzConnect:TerminalBlock_MetzConnect_Type055_RT01502HDWU_1x02_P5.00mm_Horizontal, F.Cu at (252.5, 31.5)
- added R1: 270, Resistor_THT:R_Axial_DIN0207_L6.3mm_D2.5mm_P15.24mm_Horizontal, F.Cu at (37.4, 127.0)
- added R1: 270, Resistor_THT:R_Axial_DIN0207_L6.3mm_D2.5mm_P15.24mm_Horizontal, F.Cu at (222.4, 126.5)
- added R1: 270, Resistor_THT:R_Axial_DIN0207_L6.3mm_D2.5mm_P15.24mm_Horizontal, F.Cu at (223.4, 60.5)
- added R1: 270, Resistor_THT:R_Axial_DIN0207_L6.3mm_D2.5mm_P15.24mm_Horizontal, F.Cu at (36.9, 182.5)
- added R1: 270, Resistor_THT:R_Axial_DIN0207_L6.3mm_D2.5mm_P15.24mm_Horizontal, F.Cu at (128.9, 127.0)
- added R1: 270, Resistor_THT:R_Axial_DIN0207_L6.3mm_D2.5mm_P15.24mm_Horizontal, F.Cu at (37.4, 62.0)
- added R1: 270, Resistor_THT:R_Axial_DIN0207_L6.3mm_D2.5mm_P15.24mm_Horizontal, F.Cu at (131.5, 61.4)
- added R2: 2200, Resistor_THT:R_Axial_DIN0207_L6.3mm_D2.5mm_P15.24mm_Horizontal, F.Cu at (52.6, 58.0)
- added R2: 2200, Resistor_THT:R_Axial_DIN0207_L6.3mm_D2.5mm_P15.24mm_Horizontal, F.Cu at (52.1, 178.5)
- added R2: 2200, Resistor_THT:R_Axial_DIN0207_L6.3mm_D2.5mm_P15.24mm_Horizontal, F.Cu at (144.1, 123.0)
- added R2: 2200, Resistor_THT:R_Axial_DIN0207_L6.3mm_D2.5mm_P15.24mm_Horizontal, F.Cu at (237.6, 122.5)
- added R2: 2200, Resistor_THT:R_Axial_DIN0207_L6.3mm_D2.5mm_P15.24mm_Horizontal, F.Cu at (146.7, 57.4)
- added R2: 2200, Resistor_THT:R_Axial_DIN0207_L6.3mm_D2.5mm_P15.24mm_Horizontal, F.Cu at (238.6, 56.5)
- added R2: 2200, Resistor_THT:R_Axial_DIN0207_L6.3mm_D2.5mm_P15.24mm_Horizontal, F.Cu at (52.6, 123.0)
- added RV1: 10k, Potentiometer_THT:Potentiometer_Piher_PC-16_Single_Horizontal, F.Cu at (249.0, 135.0)
- added RV1: 10k, Potentiometer_THT:Potentiometer_Piher_PC-16_Single_Horizontal, F.Cu at (63.5, 191.0)
- added RV1: 10k, Potentiometer_THT:Potentiometer_Piher_PC-16_Single_Horizontal, F.Cu at (64.0, 135.5)
- added RV1: 10k, Potentiometer_THT:Potentiometer_Piher_PC-16_Single_Horizontal, F.Cu at (158.1, 69.9)
- added RV1: 10k, Potentiometer_THT:Potentiometer_Piher_PC-16_Single_Horizontal, F.Cu at (155.5, 135.5)
- added RV1: 10k, Potentiometer_THT:Potentiometer_Piher_PC-16_Single_Horizontal, F.Cu at (250.0, 69.0)
- added RV1: 10k, Potentiometer_THT:Potentiometer_Piher_PC-16_Single_Horizontal, F.Cu at (64.0, 70.5)
- added U1: LM317_TO-220, Package_TO_SOT_THT:TO-220-3_Vertical, F.Cu at (237.0, 134.0)
- added U1: LM317_TO-220, Package_TO_SOT_THT:TO-220-3_Vertical, F.Cu at (146.1, 68.9)
- added U1: LM317_TO-220, Package_TO_SOT_THT:TO-220-3_Vertical, F.Cu at (143.5, 134.5)
- added U1: LM317_TO-220, Package_TO_SOT_THT:TO-220-3_Vertical, F.Cu at (52.0, 69.5)
- added U1: LM317_TO-220, Package_TO_SOT_THT:TO-220-3_Vertical, F.Cu at (51.5, 190.0)
- added U1: LM317_TO-220, Package_TO_SOT_THT:TO-220-3_Vertical, F.Cu at (238.0, 68.0)
- added U1: LM317_TO-220, Package_TO_SOT_THT:TO-220-3_Vertical, F.Cu at (52.0, 134.5)
- added U3: LM7805_TO220, Package_TO_SOT_THT:TO-220-3_Vertical, F.Cu at (62.0, 160.9)
- added U3: LM7805_TO220, Package_TO_SOT_THT:TO-220-3_Vertical, F.Cu at (62.5, 40.4)
- added U3: LM7805_TO220, Package_TO_SOT_THT:TO-220-3_Vertical, F.Cu at (62.5, 105.4)
- added U3: LM7805_TO220, Package_TO_SOT_THT:TO-220-3_Vertical, F.Cu at (156.6, 39.8)
- added U3: LM7805_TO220, Package_TO_SOT_THT:TO-220-3_Vertical, F.Cu at (248.5, 38.9)
- added U3: LM7805_TO220, Package_TO_SOT_THT:TO-220-3_Vertical, F.Cu at (247.5, 104.9)
- added U3: LM7805_TO220, Package_TO_SOT_THT:TO-220-3_Vertical, F.Cu at (154.0, 105.4)
Routing:
- net GND: track 144.4 -> 951.7 mm
- net Net-(D1-A): track 71.4 -> 739.0 mm
- net Net-(D1-K): track 126.0 -> 697.2 mm
- net Net-(D2-A): track 102.9 -> 408.0 mm
- net Net-(J3-Pin_1): track 0.00 -> 140.3 mm
- net Net-(J1-Pin_2): track 20.6 -> 92.1 mm
- net Net-(J1-Pin_1): track 30.7 -> 92.1 mm
- added copper zone on B.Cu, net GND
Other:
- board size 50 x 50 mm -> 236.5 x 172 mm
- board text added: "MORLET SOLUTIONS"
