File: VSource.kicad_sch (KiCad schematic)
At the start: 11 parts, among them J2 Conn_01x03_Socket, U1 LM317_TO-220

Commit message: footprints and routing
Parts:
- removed J2: Conn_01x03_Socket, symbol Connector:Conn_01x03_Socket
- added J1, J2: - +, TerminalBlock_Phoenix:TerminalBlock_Phoenix_MKDS-1,5-2-5.08_1x02_P5.08mm_Horizontal, symbol Connector_Generic:Conn_01x02
- C1: footprint (none) -> Capacitor_THT:CP_Radial_Tantal_D4.5mm_P2.50mm
- C2: footprint (none) -> Capacitor_THT:CP_Radial_D4.0mm_P2.00mm
- C3: value 4400uF -> 4700uF; footprint (none) -> Capacitor_THT:CP_Radial_D18.0mm_P7.50mm
- D1, D2: value 1N4002 -> 1N4007
- R1, R2: footprint (none) -> Resistor_THT:R_Axial_DIN0207_L6.3mm_D2.5mm_P15.24mm_Horizontal
- RV1: footprint (none) -> Potentiometer_THT:Potentiometer_Piher_PC-16_Single_Horizontal
Connections:
- net GND: now also J2.2 (Pin_2)
- net at D3.2: now also J1.2 (Pin_2)
- net at D3.3: now also J1.1 (Pin_1)
- net at C1.1, D1.2 (A), D2.1 (K)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: now also J2.1 (Pin_1)

Commit message: 5v output
Parts:
- added C4: 0.33uF, Capacitor_THT:CP_Radial_Tantal_D5.0mm_P2.50mm, symbol Device:C
- added C5: 0.1uF, Capacitor_THT:CP_Radial_Tantal_D5.0mm_P2.50mm, symbol Device:C
- added J3: - +, TerminalBlock_MetzConnect:TerminalBlock_MetzConnect_Type055_RT01502HDWU_1x02_P5.00mm_Horizontal, symbol Connector_Generic:Conn_01x02
- added U3: LM7805_TO220, Package_TO_SOT_THT:TO-220-3_Vertical, symbol Regulator_Linear:LM7805_TO220
- J1, J2: footprint TerminalBlock_Phoenix:TerminalBlock_Phoenix_MKDS-1,5-2-5.08_1x02_P5.08mm_Horizontal -> TerminalBlock_MetzConnect:TerminalBlock_MetzConnect_Type055_RT01502HDWU_1x02_P5.00mm_Horizontal
Connections:
- net GND: now also C4.2, C5.2, J3.2 (Pin_2), U3.2 (GND)
- net at C3.1, D1.1 (K), D3.4 (+)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: now also C4.1, U3.1 (VI)
- new net: C5.1, J3.1 (Pin_1), U3.3 (VO)
